File: EuroBoard/EuroBoard.kicad_sch (KiCad schematic)
At the start: 35 parts, among them J1 GPIO, J10 PD1, J11 PD2, J12 PD3, J2 Conn_01x07_Male, J3 I2C, J4 Conn_01x05_Male, J5 RX, J6 TX, J7 GND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

Commit message: Removed unnecessary caps
Parts:
- removed C4: 4.7u, Capacitor_SMD:C_0805_2012Metric_Pad1.18x1.45mm_HandSolder, symbol Device:C
- removed C5: 1u, Capacitor_SMD:C_0805_2012Metric_Pad1.18x1.45mm_HandSolder, symbol Device:C
- C6: value 4.7u -> 10u
Changed lines of the file:
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@@
   (junction (at 210.82 93.98) (diameter 0) (color 0 0 0 0)
   )
-  (junction (at 173.99 22.86) (diameter 0) (color 0 0 0 0)
-  )
   (junction (at 162.56 22.86) (diameter 0) (color 0 0 0 0)
   )
@@
     (stroke (width 0) (type default) (color 0 0 0 0))
   )
-  (wire (pts (xy 262.89 39.37) (xy 262.89 43.18))
-    (stroke (width 0) (type default) (color 0 0 0 0))
-  )
   (wire (pts (xy 177.8 113.03) (xy 172.72 113.03))
     (stroke (width 0) (type default) (color 0 0 0 0))
@@
     (stroke (width 0) (type default) (color 0 0 0 0))
   )
-  (wire (pts (xy 173.99 35.56) (xy 173.99 33.02))
-    (stroke (width 0) (type default) (color 0 0 0 0))
-  )
   (wire (pts (xy 248.92 93.98) (xy 246.38 93.98))
     (stroke (width 0) (type default) (color 0 0 0 0))
@@
     (stroke (width 0) (type default) (color 0 0 0 0))
   )
-  (wire (pts (xy 262.89 26.67) (xy 262.89 31.75))
-    (stroke (width 0) (type default) (color 0 0 0 0))
-  )
   (wire (pts (xy 147.32 46.99) (xy 147.32 52.07))
     (stroke (width 0) (type default) (color 0 0 0 0))
@@
     (stroke (width 0) (type default) (color 0 0 0 0))
   )
-  (wire (pts (xy 181.61 22.86) (xy 173.99 22.86))
-    (stroke (width 0) (type default) (color 0 0 0 0))
-  )
   (wire (pts (xy 45.72 88.9) (xy 45.72 83.82))
     (stroke (width 0) (type default) (color 0 0 0 0))
@@
     (stroke (width 0) (type default) (color 0 0 0 0))
   )
-  (wire (pts (xy 162.56 22.86) (xy 173.99 22.86))
+  (wire (pts (xy 162.56 22.86) (xy 181.61 22.86))
     (stroke (width 0) (type default) (color 0 0 0 0))
   )
@@
   )
   (wire (pts (xy 64.77 157.48) (xy 74.93 157.48))
-    (stroke (width 0) (type default) (color 0 0 0 0))
-  )
-  (wire (pts (xy 173.99 22.86) (xy 173.99 25.4))
     (stroke (width 0) (type default) (color 0 0 0 0))
   )
@@
     )
     (property "Datasheet" "~" (id 3) (at 102.87 71.12 0)
-      (effects (font (size 1.27 1.27)) hide)
-    )
-    (pin "1")
-    (pin "2")
-  )
-  (symbol (lib_id "Device:C") (at 262.89 35.56 0) (unit 1)
-    (in_bom yes) (on_board yes) (fields_autoplaced)
-    (property "Reference" "C4" (id 0) (at 266.7 34.2899 0)
-      (effects (font (size 1.27 1.27)) (justify left))
-    )
-    (property "Value" "4.7u" (id 1) (at 266.7 36.8299 0)
-      (effects (font (size 1.27 1.27)) (justify left))
-    )
-    (property "Footprint" "Capacitor_SMD:C_0805_2012Metric_Pad1.18x1.45mm_HandSolder" (id 2) (at 263.8552 39.37 0)
-      (effects (font (size 1.27 1.27)) hide)
-    )
-    (property "Datasheet" "~" (id 3) (at 262.89 35.56 0)
       (effects (font (size 1.27 1.27)) hide)
     )
@@
     (pin "1")
   )
-  (symbol (lib_id "Device:C") (at 173.99 29.21 0) (unit 1)
-    (in_bom yes) (on_board yes) (fields_autoplaced)
-    (property "Reference" "C5" (id 0) (at 177.8 27.9399 0)
-      (effects (font (size 1.27 1.27)) (justify left))
-    )
-    (property "Value" "1u" (id 1) (at 177.8 30.4799 0)
-      (effects (font (size 1.27 1.27)) (justify left))
-    )
-    (property "Footprint" "Capacitor_SMD:C_0805_2012Metric_Pad1.18x1.45mm_HandSolder" (id 2) (at 174.9552 33.02 0)
-      (effects (font (size 1.27 1.27)) hide)
-    )
-    (property "Datasheet" "~" (id 3) (at 173.99 29.21 0)
-      (effects (font (size 1.27 1.27)) hide)
-    )
-    (pin "1")
-    (pin "2")
-  )
   (symbol (lib_id "power:+5V") (at 97.79 140.97 270) (unit 1)
     (in_bom yes) (on_board yes) (fields_autoplaced)
@@
     (pin "1")
   )
-  (symbol (lib_id "power:GND") (at 262.89 43.18 0) (unit 1)
-    (in_bom yes) (on_board yes) (fields_autoplaced)
-    (property "Reference" "#PWR0108" (id 0) (at 262.89 49.53 0)
-      (effects (font (size 1.27 1.27)) hide)
-    )
-    (property "Value" "GND" (id 1) (at 262.89 48.26 0))
-    (property "Footprint" "" (id 2) (at 262.89 43.18 0)
-      (effects (font (size 1.27 1.27)) hide)
-    )
-    (property "Datasheet" "" (id 3) (at 262.89 43.18 0)
-      (effects (font (size 1.27 1.27)) hide)
-    )
-    (pin "1")
-  )
   (symbol (lib_id "power:+12V") (at 97.79 143.51 270) (unit 1)
     (in_bom yes) (on_board yes) (fields_autoplaced)
@@
     )
     (property "Datasheet" "" (id 3) (at 97.79 138.43 0)
-      (effects (font (size 1.27 1.27)) hide)
-    )
-    (pin "1")
-  )
-  (symbol (lib_id "power:GND") (at 173.99 35.56 0) (unit 1)
-    (in_bom yes) (on_board yes) (fields_autoplaced)
-    (property "Reference" "#PWR0110" (id 0) (at 173.99 41.91 0)
-      (effects (font (size 1.27 1.27)) hide)
-    )
-    (property "Value" "GND" (id 1) (at 173.99 40.64 0))
-    (property "Footprint" "" (id 2) (at 173.99 35.56 0)
-      (effects (font (size 1.27 1.27)) hide)
-    )
-    (property "Datasheet" "" (id 3) (at 173.99 35.56 0)
       (effects (font (size 1.27 1.27)) hide)
     )
@@
       (effects (font (size 1.27 1.27)) (justify left))
     )
-    (property "Value" "4.7u" (id 1) (at 207.01 30.4799 0)
+    (property "Value" "10u" (id 1) (at 207.01 30.4799 0)
       (effects (font (size 1.27 1.27)) (justify left))
     )
@@
     (pin "1")
   )
-  (symbol (lib_id "power:+3.3V") (at 262.89 26.67 0) (unit 1)
-    (in_bom yes) (on_board yes) (fields_autoplaced)
-    (property "Reference" "#PWR0109" (id 0) (at 262.89 30.48 0)
-      (effects (font (size 1.27 1.27)) hide)
-    )
-    (property "Value" "+3.3V" (id 1) (at 262.89 21.59 0))
-    (property "Footprint" "" (id 2) (at 262.89 26.67 0)
-      (effects (font (size 1.27 1.27)) hide)
-    )
-    (property "Datasheet" "" (id 3) (at 262.89 26.67 0)
-      (effects (font (size 1.27 1.27)) hide)
-    )
-    (pin "1")
-  )
   (symbol (lib_id "power:GND") (at 50.8 72.39 0) (unit 1)
     (in_bom yes) (on_board yes)
@@
       (reference "#PWR0107") (unit 1) (value "+3.3V") (footprint "")
     )
-    (path "/42fd7900-552e-4642-ab60-7e30d6cd8ca2"
-      (reference "#PWR0108") (unit 1) (value "GND") (footprint "")
-    )
-    (path "/ed886fb5-fcc6-43a9-b75d-0e3c9c7569ba"
-      (reference "#PWR0109") (unit 1) (value "+3.3V") (footprint "")
-    )
-    (path "/4863f85b-d9f9-42a5-9d56-af535db8fbd9"
-      (reference "#PWR0110") (unit 1) (value "GND") (footprint "")
-    )
     (path "/ecb73b8c-3d8b-47f7-ac3c-849a31982412"
       (reference "#PWR0111") (unit 1) (value "+5V") (footprint "")
@@
       (reference "C2") (unit 1) (value "100n") (footprint "Capacitor_SMD:C_0805_2012Metric_Pad1.18x1.45mm_HandSolder")
     )
-    (path "/043b155d-617c-4e7d-823d-64db63c32c2a"
-      (reference "C4") (unit 1) (value "4.7u") (footprint "Capacitor_SMD:C_0805_2012Metric_Pad1.18x1.45mm_HandSolder")
-    )
-    (path "/4144307f-3cde-4fd1-99e5-0392d5177819"
-      (reference "C5") (unit 1) (value "1u") (footprint "Capacitor_SMD:C_0805_2012Metric_Pad1.18x1.45mm_HandSolder")
-    )
     (path "/af3713c5-ab8e-47d8-9144-f62cbe584e43"
-      (reference "C6") (unit 1) (value "4.7u") (footprint "Capacitor_SMD:C_0805_2012Metric_Pad1.18x1.45mm_HandSolder")
+      (reference "C6") (unit 1) (value "10u") (footprint "Capacitor_SMD:C_0805_2012Metric_Pad1.18x1.45mm_HandSolder")
     )
     (path "/be58abdc-63a2-4c4a-9328-a3316e736bde"
