File: Power.kicad_sch (KiCad schematic)
At the start: 7 parts, among them U301 AMS1117-3.3

Commit message: MPN and MOUSER added PSU
Parts:
- F301: MPN (none) -> 1206L050/15YR; Mouser (none) -> 576-1206L050/15YR
- U301: MPN (none) -> AZ1117IH-3.3TRG1; Mouser (none) -> 621-AZ1117IH-3.3TRG1
Changed lines of the file:
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@@
+      (effects (font (size 1.27 1.27)) hide)
+    )
+    (property "MPN" "1206L050/15YR" (at 27.94 40.64 90)
+      (effects (font (size 1.27 1.27)) hide)
+    )
+    (property "Mouser" "576-1206L050/15YR" (at 27.94 40.64 90)
       (effects (font (size 1.27 1.27)) hide)
     )
@@
       (effects (font (size 1.27 1.27)) hide)
     )
+    (property "MPN" "AZ1117IH-3.3TRG1" (at 69.85 40.64 0)
+      (effects (font (size 1.27 1.27)) hide)
+    )
+    (property "Mouser" "621-AZ1117IH-3.3TRG1" (at 69.85 40.64 0)
+      (effects (font (size 1.27 1.27)) hide)
+    )
