File: Power.kicad_sch (KiCad schematic)
At the start: 7 parts, among them U301 AMS1117-3.3

Commit message: Converted for use as the single EuroMeasure.sch file
Parts:
- removed C301, C303: 10u, Capacitor_SMD:C_0805_2012Metric_Pad1.18x1.45mm_HandSolder, symbol Device:C
- removed C302, C304: 220u, Capacitor_SMD:CP_Elec_6.3x7.7, symbol Device:C_Polarized
- removed F301: Polyfuse, Fuse:Fuse_1210_3225Metric, symbol Device:Polyfuse
- removed TP301: 3V3, MEMS_Custom:TestPoint_Pad_D1.0mm, symbol Connector:TestPoint
- removed U301: AMS1117-3.3, Package_TO_SOT_SMD:SOT-223-3_TabPin2, symbol Regulator_Linear:AMS1117-3.3
Other:
- note removed: "3V3 supply"
