File: EuroMeasure.kicad_sch (KiCad schematic)
At the start: 33 parts, among them SW1 RST, SW2 SW_DIP_x04, U3 AZ1117-3V3, U4 STM32G030CxT, Y1 16MHz

Commit message: Fixed reset pullup
Parts:
- added R2 (x2): 1k, Resistor_SMD:R_0805_2012Metric_Pad1.20x1.40mm_HandSolder, symbol Device:R_Small
- renumbered C1 to C2, C13 to C24, C12 to C25, C16 to C26, C14 to C27, C21 to C41, C20 to C44, C23 to C52, C25 to C53, C24 to C54, D6 to D1, D14 to D7, F2 to F3, JP1 to JP15, JP4 to JP16, JP3 to JP17, JP2 to JP18, L3 to L1, R21 to R19, R9 to R2, R23 to R33, R20 to R34, TP13 to TP10, TP12 to TP11, TP2 to TP4, TP1 to TP5, TP11 to TP6, U3 to U5, U4 to U9
Connections:
- net +3.3V: now also R2.2
- net RST_LOCAL: now also R2.1, R2.1; no longer D7.2 (A)
- net 5v_fused: no longer names the net of C25.1, C27.1, F3.2, U5.3 (VI)
- net led_r: no longer names the net of D1.2 (A), R2.1
- net osc_mid: no longer names the net of C44.1, R33.1, Y1.1
- new net: D7.2 (A), R2.2
Other:
- moved on the sheet: D7

Commit message: Edited visibility in bom
Parts:
- JP1: renamed from JP17; now left out of the parts list
- JP2: renamed from JP15; now left out of the parts list
- JP3: renamed from JP16; now left out of the parts list
- JP4: renamed from JP18; now left out of the parts list
- TP10: renamed from TP5; symbol Connector:TestPoint -> MEMS_Electromechanical:TestPoint; now left out of the parts list
- TP6: renamed from TP11; symbol Connector:TestPoint -> MEMS_Electromechanical:TestPoint; now left out of the parts list
- TP7: renamed from TP10; symbol Connector:TestPoint -> MEMS_Electromechanical:TestPoint; now left out of the parts list
- TP8: renamed from TP4; symbol Connector:TestPoint -> MEMS_Electromechanical:TestPoint; now left out of the parts list
- TP9: renamed from TP6; symbol Connector:TestPoint -> MEMS_Electromechanical:TestPoint; now left out of the parts list
- renumbered C27 to C1, C54 to C10, C25 to C2, C24 to C3, C26 to C4, C2 to C5, C41 to C6, C44 to C7, C52 to C8, C53 to C9, D7 to D1, D1 to D2, F3 to F1, R19 to R1, R34 to R2, R33 to R3, R2 to R4, R2 to R5, R2 to R6, SW2 to SW1, SW1 to SW2, U5 to U1, U9 to U2
